File: Can_Board/CAN_Board.sch (EAGLE design)
At the start: 18 parts, among them J1 22-05-7028-02, J2 22-05-7028-02, U11 MCP2561-E/SN, X1 MSTBA2, X11 5504F1-09S-02A-03

Commit message: Route the board
Parts:
- removed JP5: FIDUCIAL1X2, SparkFun:FIDUCIAL1X2
- removed X11: 5504F1-09S-02A-03, con-multicomp:5504F1-09S-02A-03
- added J3: 22-05-7028-02, con-molex:22-05-7028-02
- added JP3: FIDUCIAL1X2, SparkFun:FIDUCIAL1X2
- J2: value 22-05-7028-02 -> 5504F1-09S-02A-03; device con-molex:22-05-7028-02 -> con-multicomp:5504F1-09S-02A-03
- renumbered C13 to C1, C136 to C2, R54 to R2, R55 to R1, U$2 to T1, U11 to U1
Connections:
- net +24V: now also J2C.9; no longer X11C.9
- net +3V3: now also J1-1.S; no longer J1-2.S
- net CAN_N: now also J2C.2; no longer X11C.2
- net CAN_P: now also J2C.7; no longer X11C.7
- net CAN_RX: now also J3-1.S; no longer J2-1.S
- net CAN_SHLD: now also J2C.5; no longer X11C.5
- net CAN_TX: now also J3-2.S; no longer J2-2.S
- net GND: now also J1-2.S, J2C.3, J2C.6; no longer J1-1.S, X11C.3, X11C.6
Other:
- moved on the sheet: J1-1, J1-2, X1-1, X1-2

Commit message: Update components names and value placement
Parts:
- C1: MPN (none) -> MC0603B472K500CT; OC_NEWARK (none) -> 33R0458
- C2: MPN (none) -> MC0603B104K250CT; OC_NEWARK (none) -> 06R4925
- H1, H2, H3, H4, JP1, JP2, JP3, JP4, T1: OC_NEWARK (none) -> unknown
- J1, J3: MPN (none) -> 22-05-7028; OC_NEWARK (none) -> 25M1728
- J2: MPN (none) -> 5504F1-09S-02A-03; OC_NEWARK (none) -> 18T0703
- R1, R2: MPN (none) -> MCMR06X60R4FTL; OC_NEWARK (none) -> 86T3680
- U1: MPN (none) -> MCP2561-E/SN; OC_NEWARK (none) -> 12X8698
