File: MCU_Board/MCU_Board.brd (EAGLE design)
At the start: 83 x 41 mm, 81 parts, among them J1 22-05-7068-06, J10 22-27-2061-06, J11 22-05-7068-06, J12 22-05-7048-04, J13 22-05-7048-04, J2 22-05-7068-06, J3 22-05-7028-02, J4 22-05-7028-02, J5 22-05-7038-03, J6 22-05-7048-04, J7 22-05-7048-04, J8 22-05-7038-03, J9 22-05-7028-02, SW1 B3FS-1015, SW2 B3FS-1015, T1 MMBT2222AL, U2 TPL0401A, U3 SN74LVC3G17DCTR, U4 SN74LVC3G17DCTR, U7 LPC1768FBD100, U8 AT24C512C-SSHM-B, X6 USB3075-30-A, X9 1241050-5

Commit message: Route the MCU board
Parts:
- removed C101, C102, C103, C104, C105, C106, C107, C108, C109, C111, C115, C118, C119, C123, C124, C125, C126: 0.1uF, rcl:C0603
- removed C121: 10uF, rcl:CT3216
- removed C127, C128: 18pF, rcl:C0603
- removed JP3: BC-2-P, exmachina:BC-2-P
- removed L100: 0603PS-103KLB, coilcraft:0603
- removed LED5: (no value), led:CHIPLED_0603
- removed R100, R101: 0R, rcl:R0603
- removed R102, R103: 10K, rcl:R0603
- removed R29, R30, R33: 4K7, rcl:R0603
- removed R35, R36: 33, rcl:R0603
- removed R38, R39: 1K5, rcl:R0603
- removed U$1: 3000, keystone:3000
- removed U7: LPC1768FBD100, NXP:SOT407-1
- removed U8: AT24C512C-SSHM-B, atmel:SOIC127P600X175-8N
- removed X6: USB3075-30-A, con-GlobalConnectorTechnology:USB_MICROB_SMT
- removed X9: 1241050-5, con-amp:2.54/2X5
- removed XT2: FC-135, crystal:FC-135
- removed XT3: ASE-12, crystal:ASE
- added C1: 10uF, rcl:CT3216
- added C10, C5: 18pF, rcl:C0603
- added C11, C13, C14, C15, C16, C17, C18, C19, C2, C20, C21, C3, C4, C6, C7, C8, C9: 0.1uF, rcl:C0603
- added J14: 22-05-7048-04, con-molex:7395-04
- added J15: 1241050-5, con-amp:2.54/2X5
- added JP1: BC-2-P, exmachina:BC-2-P
- added L1: 0603PS-103KLB, coilcraft:0603
- added LED1: (no value), led:CHIPLED_0603
- added R1: 4K7, rcl:R0603
- added R18, R19, R20, R21, R22, R23: 1K, rcl:R0603
- added R24, R25, R26, R27: 100, rcl:R0603
- added U1: AT24C512C-SSHM-B, atmel:SOIC127P600X175-8N
- added U5: SN74LVC3G17DCTR, ti:SOP65P400X130-8N
- added X1: FC-135, crystal:FC-135
- added X2: ASE-12, crystal:ASE
- added X3: 3000, keystone:3000
- J10: value 22-27-2061-06 -> 22-05-7068-06; device con-molex:6410-06 -> con-molex:7395-06
- J11: value 22-05-7068-06 -> 22-05-7048-04; device con-molex:7395-06 -> con-molex:7395-04
- J12: value 22-05-7048-04 -> 22-27-2061-06; device con-molex:7395-04 -> con-molex:6410-06
- J13: value 22-05-7048-04 -> USB3075-30-A; device con-molex:7395-04 -> con-GlobalConnectorTechnology:USB_MICROB_SMT
- J7: value 22-05-7048-04 -> 22-05-7038-03; device con-molex:7395-04 -> con-molex:7395-03
- J8: value 22-05-7038-03 -> 22-05-7048-04; device con-molex:7395-03 -> con-molex:7395-04
- R10, R12: value 1K -> 4K7
- R11: value 1K -> 33
- R13: value 1K -> 100
- R14: value 4K7 -> 1K5
- R15: value 100 -> 33
- R16: value 0R -> 33
- R17: value 0R -> 1K5
- R3: value 33 -> 4K7
- R4, R5: value 100 -> 0R
- R6, R7: value 100 -> 10K
- R8, R9: value 1K -> 0R
- U2: value TPL0401A -> LPC1768FBD100; device ti:SC-70-DCK -> NXP:SOT407-1
- U3: value SN74LVC3G17DCTR -> TPL0401A; device ti:SOP65P400X130-8N -> ti:SC-70-DCK
- moved J8 79.6 mm to (81.2, 35.6), turned to 180 degrees
- moved J13 77.2 mm to (1.44, 11.8), turned to 270 degrees
- moved SW1 71.3 mm to (81.3, 22.4), turned to 0 degrees
- moved J7 44.5 mm to (12.6, 5.08)
- moved J10 35.6 mm to (49.5, 5.08), turned to 0 degrees
- moved J12 33.2 mm to (8.21, 28.4), turned to 180 degrees
- moved R12 30.2 mm to (35.0, 7.62), flipped to the bottom
- moved R15 28.5 mm to (7.79, 13.1), flipped to the top
- moved R14 25.6 mm to (11.0, 8.64), flipped to the top, turned to 0 degrees
- moved R10 25.0 mm to (38.8, 7.62), flipped to the bottom, turned to 0 degrees
- moved R7 21.7 mm to (74.8, 9.91), flipped to the top, turned to 270 degrees
- moved U3 21.2 mm to (36.9, 9.65), flipped to the bottom, turned to 270 degrees
- moved R16 19.6 mm to (7.79, 10.9), turned to 0 degrees
- moved U2 19.4 mm to (46.9, 20.3), flipped to the top, turned to 0 degrees
- moved T1 17.4 mm to (53.5, 13.1)
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Connections:
- new net ETH_RST: J1.6, U2.44
- new net ETH_X1: J1.1, U2.88
- net +3V3: now also C1.+, C11.1, C2.1, C20.1, C21.1, C3.1, C4.1, C6.1, C7.1, C8.1, J15.1, L1.P$1, LED1.A, R1.2, R10.1, R12.1, R17.1, R2.2, R3.2, R6.2, R7.2, U1.8, U2.13, U2.28, U2.42, U2.54, U2.71, U2.84, U2.96, U5.8, X2.1, X2.4; no longer C108.1, C109.1, C111.1, C115.1, C118.1, C119.1, C121.+, C123.1, C124.1, C125.1, L100.P$1, LED5.A, R102.2, R103.2, R14.1, R2.1, R29.2, R30.2, R33.2, R38.1, U3.8, U7.13, U7.28, U7.42, U7.54, U7.71, U7.84, U7.96, U8.8, X9.1, XT3.1, XT3.4
- net +5V: now also C13.1, R11.1, U3.1, U3.6; no longer C101.1, R3.1, U2.1, U2.6
- net ADC_SLACK_DETECTION: now also U2.7; no longer U7.7
- net ADC_TEMP_0: now also U2.9; no longer U7.9
- net ADC_TEMP_1: now also U2.8; no longer U7.8
- net AVDD: now also C9.1, L1.P$2, U2.10, U2.12; no longer C126.1, L100.P$2, U7.10, U7.12
- net BOOT_SELECT_P2_10: now also R8.1, U2.53; no longer R100.1, U7.53
- net BOOT_SELECT_P2_12: now also R9.1, U2.51; no longer R101.1, U7.51
- net BRAKE_SENSOR_1: now also U2.81; no longer U7.81
- net BRAKE_SENSOR_2: now also U2.80; no longer U7.80
- net CAN_RX: now also U2.46; no longer U7.46
- net CAN_TX: now also U2.47; no longer U7.47
- net DRIVE_EN: now also U2.79; no longer U7.79
- net DRIVE_ERR: now also U2.78; no longer U7.78
- net EEPROM_SCL: now also R3.1, U1.6, U2.24; no longer R30.1, U7.24, U8.6
- net EEPROM_SDA: now also R2.1, U1.5, U2.25; no longer R33.1, U7.25, U8.5
- net ENCODER_A: now also J7.1, U2.34; no longer J8.1, U7.34
- net ENCODER_B: now also J7.2, U2.37; no longer J8.2, U7.37
- net ENCODER_Z: now also J7.3, U2.38; no longer J8.3, U7.38
- net ETH_CLK_EN: now also U2.43; no longer U7.43
- net ETH_CRS: now also U2.92; no longer U7.92
- net ETH_MDC: now also U2.87; no longer U7.87
- net ETH_MDIO: now also U2.86; no longer U7.86
- net ETH_RXD_0: now also U2.91; no longer U7.91
- net ETH_RXD_1: now also U2.90; no longer U7.90
- net ETH_RX_ER: now also U2.89; no longer U7.89
- net ETH_TXD_0: now also U2.95; no longer U7.95
- net ETH_TXD_1: now also U2.94; no longer U7.94
- net ETH_TXD_EN: now also U2.93; no longer U7.93
- net FAN_1_PWM: now also J8.1, U2.75; no longer J7.1, U7.75
- net FAN_1_SENSOR: now also J8.2, U2.77; no longer J7.2, U7.77
- net FAN_2_PWM: now also J8.3, U2.74; no longer J7.3, U7.74
- net FAN_2_SENSOR: now also J8.4, U2.76; no longer J7.4, U7.76
- net GND: now also C1.-, C10.2, C11.2, C13.2, C14.2, C15.2, C16.2, C17.2, C18.2, C19.2, C2.2, C20.2, C21.2, C3.2, C4.2, C5.2, C6.2, C7.2, C8.2, C9.2, J1.2, J12.1, J13.5, J15.2, JP1.2, U1.1, U1.2, U1.3, U1.4, U2.11, U2.15, U2.31, U2.41, U2.55, U2.72, U2.83, U2.97, U3.2, U5.4, X2.2, X3.-; no longer C101.2, C102.2, C103.2, C104.2, C105.2, C106.2, C107.2, C108.2, C109.2, C111.2, C115.2, C118.2, C119.2, C121.-, C123.2, C124.2, C125.2, C126.2, C127.2, C128.2, JP3.2, U$1.-, U2.2, U3.4, U7.11, U7.15, U7.31, U7.41, U7.55, U7.72, U7.83, U7.97, U8.1, U8.2, U8.3, U8.4, X6.5, X9.2, XT3.2
- net HMI_BUTTON_1: now also J10.1, R18.1; no longer J11.1, R13.1
- net HMI_BUTTON_2: now also J10.2, R19.1; no longer J11.2, R12.1
- net HMI_BUTTON_3: now also J10.3, R20.1; no longer J11.3, R11.1
- net HMI_BUTTON_4: now also J10.4, R21.1; no longer J11.4, R10.1
- net HMI_BUTTON_5: now also J10.5, R22.1; no longer J11.5, R9.1
- net HMI_BUTTON_6: now also J10.6, R23.1; no longer J11.6, R8.1
- net HMI_BUTTON_CPU_1: now also U2.63; no longer U7.63
- net HMI_BUTTON_CPU_2: now also U2.62; no longer U7.62
- net HMI_BUTTON_CPU_3: now also U2.61; no longer U7.61
- net HMI_BUTTON_CPU_4: now also U2.60, U5.1; no longer U3.1, U7.60
- net HMI_BUTTON_CPU_5: now also U2.59, U5.3; no longer U3.3, U7.59
- net HMI_BUTTON_CPU_6: now also R4.2, R5.1, U5.6; no longer R16.2, R17.1, U3.6
- net HMI_BUTTON_MCU_FCT_6: now also R5.2, U2.58; no longer R17.2, U7.58
- net HMI_LCD_BACKLIGHT: now also R13.2, U2.56; no longer R15.2, U7.56
- net HMI_LCD_LED+: now also J11.1, R11.2; no longer J12.1, R3.2
- net HMI_LCD_SCL: now also J11.2, R10.2, U2.49, U3.3; no longer J12.2, R14.2, U2.3, U7.49
- net HMI_LCD_SDA: now also J11.3, R12.2, U2.48, U3.4; no longer J12.3, R2.2, U2.4, U7.48
- net HMI_LCD_VO: now also J11.4, U3.5; no longer J12.4, U2.5
- net HMI_LED_1: now also R24.1, U2.73; no longer R7.1, U7.73
- net HMI_LED_2: now also R25.2, U2.70; no longer R6.2, U7.70
- net HMI_LED_3: now also R26.1, U2.69; no longer R5.1, U7.69
- net HMI_LED_4: now also R27.2, U2.68; no longer R4.2, U7.68
- net ISP_RXDO: now also J12.4, J15.3, U2.99; no longer U7.99, X9.3
- net ISP_TXDO: now also J12.5, J15.4, U2.98; no longer U7.98, X9.4
- net JTAG_TCK: now also J15.8, U2.5; no longer U7.5, X9.8
- net JTAG_TDI: now also J15.7, U2.2; no longer U7.2, X9.7
- net JTAG_TDO: now also J15.9, U2.1; no longer U7.1, X9.9
- net JTAG_TMS: now also J15.10, U2.3; no longer U7.3, X9.10
- net N$1: now also J14.2, R25.1; no longer J13.2, R6.1
- net N$15: now also J13.2, R15.1, R17.2; no longer R36.1, R38.2, X6.2
- net N$16: now also J13.3, R16.1; no longer R35.1, X6.3
- net N$17: now also C14.1, R18.2; no longer C102.1, R13.2
- net N$18: now also LED1.C, R14.1; no longer LED5.C, R39.1
- net N$19: now also C16.1, R19.2; no longer C103.1, R12.2
- net N$2: now also J14.4, R27.1; no longer J13.4, R4.1
- net N$20: now also C18.1, R20.2; no longer C104.1, R11.2
- net N$22: now also JP1.1, R1.1, U1.7; no longer JP3.1, R29.1, U8.7
- net N$25: now also C15.1, R21.2, U5.7; no longer C105.1, R10.2, U3.7
- net N$26: now also C17.1, R22.2, U5.5; no longer C106.1, R9.2, U3.5
- net N$27: now also C19.1, R23.2, U5.2; no longer C107.1, R8.2, U3.2
- net N$5: now also R7.1, R8.2, R9.2; no longer R100.2, R101.2, R102.1
- net N$63: now also J14.1, R24.2; no longer J13.1, R7.2
- net N$64: now also J14.3, R26.2; no longer J13.3, R5.2
- net N$7: now also R13.1; no longer R15.1
- net RESET: now also J15.5, R4.1, R6.1, U2.17; no longer R103.1, R16.1, U7.17, X9.5
- net RTCX1: now also C5.1, U2.16, X1.1; no longer C127.1, U7.16, XT2.1
- net RTCX2: now also C10.1, U2.18, X1.2; no longer C128.1, U7.18, XT2.2
- net USB_D_N: now also R16.2, U2.30; no longer R35.2, U7.30
- net USB_D_P: now also R15.2, U2.29; no longer R36.2, U7.29
- net USB_UP_LED: now also R14.2, U2.32; no longer R39.2, U7.32
- net USB_V_BUS: now also J13.1, U2.21; no longer U7.21, X6.1
- net VBAT+: now also U2.19, X3.+1, X3.+2; no longer U$1.+1, U$1.+2, U7.19
- net XTAL1: now also U2.22, X2.3; no longer U7.22, XT3.3
Routing:
- net RESET: track 0.00 -> 105.9 mm, vias 0 -> 3
- net VBAT+: track 0.00 -> 83.9 mm, vias 0 -> 3
- net +5V: track 0.00 -> 74.7 mm, vias 0 -> 3
- net +3V3: track 0.00 -> 57.0 mm, vias 0 -> 33
- net ISP_TXDO: track 0.00 -> 48.0 mm, vias 0 -> 1
- net ISP_RXDO: track 0.00 -> 47.4 mm, vias 0 -> 1
- net ENCODER_Z: track 1.27 -> 46.2 mm, vias 0 -> 1
- net ADC_TEMP_0: track 0.00 -> 40.1 mm
- net HMI_BUTTON_MCU_FCT_6: track 0.00 -> 39.3 mm, vias 0 -> 4
- net ENCODER_B: track 2.79 -> 41.8 mm, vias 0 -> 1
- net USB_V_BUS: track 0.00 -> 37.9 mm, vias 0 -> 2
- net ADC_TEMP_1: track 0.00 -> 37.3 mm
- net JTAG_TCK: track 0.00 -> 37.0 mm, vias 0 -> 2
- net USB_UP_LED: track 0.00 -> 36.9 mm, vias 0 -> 2
- net FAN_2_SENSOR: track 0.00 -> 36.7 mm, vias 0 -> 1
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- added copper zone on layer 15, net +3V3
- added copper zone on layer 16, net GND
- added copper zone on layer 2, net GND
Other:
- board size 83 x 41 mm -> 88 x 41 mm
