File: MCU_Board/MCU_Board.sch (EAGLE design)
At the start: 81 parts, among them J1 22-05-7068-06, J10 22-27-2061-06, J11 22-05-7068-06, J12 22-05-7048-04, J13 22-05-7048-04, J2 22-05-7068-06, J3 22-05-7028-02, J4 22-05-7028-02, J5 22-05-7038-03, J6 22-05-7048-04, J7 22-05-7048-04, J8 22-05-7038-03, J9 22-05-7028-02, SW1 B3FS-1015, SW2 B3FS-1015, T1 MMBT2222AL, U2 TPL0401A, U3 SN74LVC3G17DCTR, U4 SN74LVC3G17DCTR, U7 LPC1768FBD100, U8 AT24C512C-SSHM-B, X6 USB3075-30-A, X9 1241050-5

Commit message: Route the MCU board
Parts:
- removed C115: 0.1uF, rcl:C-EUC0603
- removed R100, R101: 0R, rcl:R-EU_R0603
- removed R102, R103: 10K, rcl:R-EU_R0603
- removed R30, R33: 4K7, rcl:R-EU_R0603
- removed R35, R36: 33, rcl:R-EU_R0603
- removed R38, R39: 1K5, rcl:R-EU_R0603
- removed U7: LPC1768FBD100, NXP:LPC1768FBD100
- removed X6: USB3075-30-A, con-GlobalConnectorTechnology:USB3075-30-A
- added C3: 0.1uF, rcl:C-EUC0603
- added J14: 22-05-7048-04, con-molex:22-05-7048-04
- added R18, R19, R20, R21, R22, R23: 1K, rcl:R-EU_R0603
- added R24, R25, R26, R27: 100, rcl:R-EU_R0603
- added U5: SN74LVC3G17DCTR, ti:SN74LVC3G17DCTR
- J10: value 22-27-2061-06 -> 22-05-7068-06; device con-molex:22-27-2061-06 -> con-molex:22-05-7068-06
- J11: value 22-05-7068-06 -> 22-05-7048-04; device con-molex:22-05-7068-06 -> con-molex:22-05-7048-04
- J12: value 22-05-7048-04 -> 22-27-2061-06; device con-molex:22-05-7048-04 -> con-molex:22-27-2061-06
- J13: value 22-05-7048-04 -> USB3075-30-A; device con-molex:22-05-7048-04 -> con-GlobalConnectorTechnology:USB3075-30-A
- J7: value 22-05-7048-04 -> 22-05-7038-03; device con-molex:22-05-7048-04 -> con-molex:22-05-7038-03
- J8: value 22-05-7038-03 -> 22-05-7048-04; device con-molex:22-05-7038-03 -> con-molex:22-05-7048-04
- R10, R12: value 1K -> 4K7
- R11: value 1K -> 33
- R13: value 1K -> 100
- R14: value 4K7 -> 1K5
- R15: value 100 -> 33
- R16: value 0R -> 33
- R17: value 0R -> 1K5
- R3: value 33 -> 4K7
- R4, R5: value 100 -> 0R
- R6, R7: value 100 -> 10K
- R8, R9: value 1K -> 0R
- U2: value TPL0401A -> LPC1768FBD100; device ti:TPL0401A -> NXP:LPC1768FBD100
- U3: value SN74LVC3G17DCTR -> TPL0401A; device ti:SN74LVC3G17DCTR -> ti:TPL0401A
- renumbered C101 to C13, C102 to C14, C103 to C16, C104 to C18, C105 to C15, C106 to C17, C107 to C19, C108 to C20, C109 to C21, C111 to C2, C118 to C7, C119 to C11, C121 to C1, C123 to C4, C124 to C6, C125 to C8, C126 to C9, C127 to C5, C128 to C10, JP3 to JP1, L100 to L1, LED5 to LED1, R29 to R1, U$1 to X3, U8 to U1, X9 to J15, XT2 to X1, XT3 to X2
Connections:
- new net ETH_RST: J1-6.S, U2.P1[28]/MCOA2/PCAP1[0]/MAT0[0]
- new net ETH_X1: J1-1.S, U2.P1[15]/ENET_REF_CLK
- net +3V3: now also C3.1, R10.1, R12.1, R17.1, R2.2, R3.2, R6.2, R7.2, U2.NC, U2.VDD, U2.VDD_2, U2.VDD_3, U2.VDD_4, U2.VDD_5, U2.VDD_6, U5.VCC; no longer C115.1, R102.2, R103.2, R14.1, R2.1, R30.2, R33.2, R38.1, U3.VCC, U7.NC, U7.VDD, U7.VDD_2, U7.VDD_3, U7.VDD_4, U7.VDD_5, U7.VDD_6
- net +5V: now also R11.1, U3.H, U3.VDD; no longer R3.1, U2.H, U2.VDD
- net ADC_SLACK_DETECTION: now also U2.P0[25]/AD0[2]/I2SRX_SDA/TXD3; no longer U7.P0[25]/AD0[2]/I2SRX_SDA/TXD3
- net ADC_TEMP_0: now also U2.P0[23]/AD0[0]/I2SRX_CLK/CAP3[0]; no longer U7.P0[23]/AD0[0]/I2SRX_CLK/CAP3[0]
- net ADC_TEMP_1: now also U2.P0[24]/AD0[1]/I2SRX_WS/CAP3[1]; no longer U7.P0[24]/AD0[1]/I2SRX_WS/CAP3[1]
- net AVDD: now also U2.VDDA, U2.VREFP; no longer U7.VDDA, U7.VREFP
- net BOOT_SELECT_P2_10: now also R8.1, U2.P2[10]/*EINT0/NMI; no longer R100.1, U7.P2[10]/*EINT0/NMI
- net BOOT_SELECT_P2_12: now also R9.1, U2.P2[12]/*EINT2/I2STX_WS; no longer R101.1, U7.P2[12]/*EINT2/I2STX_WS
- net BRAKE_SENSOR_1: now also U2.P0[4]/I2SRX_CLK/RD2/CAP2[0]; no longer U7.P0[4]/I2SRX_CLK/RD2/CAP2[0]
- net BRAKE_SENSOR_2: now also U2.P0[5]/I2SRX_WS/TD2/CAP2[1]; no longer U7.P0[5]/I2SRX_WS/TD2/CAP2[1]
- net CAN_RX: now also U2.P0[0]/RD1/TXD3/SDA1; no longer U7.P0[0]/RD1/TXD3/SDA1
- net CAN_TX: now also U2.P0[1]/TD1/RXD3/SCL1; no longer U7.P0[1]/TD1/RXD3/SCL1
- net DRIVE_EN: now also U2.P0[6]/I2SRX_SDA/SSEL1/MAT2[0]; no longer U7.P0[6]/I2SRX_SDA/SSEL1/MAT2[0]
- net DRIVE_ERR: now also U2.P0[7]/I2STX_CLK/SCK1/MAT2[1]; no longer U7.P0[7]/I2STX_CLK/SCK1/MAT2[1]
- net EEPROM_SCL: now also R3.1, U2.P0[28]/SCL0/USB_SCL; no longer R30.1, U7.P0[28]/SCL0/USB_SCL
- net EEPROM_SDA: now also R2.1, U2.P0[27]/SDA0/USB_SDA; no longer R33.1, U7.P0[27]/SDA0/USB_SDA
- net ENCODER_A: now also J7-1.S, U2.P1[20]/MCI0/PWM1[2]/SCK0; no longer J8-1.S, U7.P1[20]/MCI0/PWM1[2]/SCK0
- net ENCODER_B: now also J7-2.S, U2.P1[23]/MCI1/PWM1[4]/MISO0; no longer J8-2.S, U7.P1[23]/MCI1/PWM1[4]/MISO0
- net ENCODER_Z: now also J7-3.S, U2.P1[24]/MCI2/PWM1[5]/MOSI0; no longer J8-3.S, U7.P1[24]/MCI2/PWM1[5]/MOSI0
- net ETH_CLK_EN: now also U2.P1[27]/CLKOUT/*USB_OVRCR/CAP0[1]; no longer U7.P1[27]/CLKOUT/*USB_OVRCR/CAP0[1]
- net ETH_CRS: now also U2.P1[8]/ENET_CRS; no longer U7.P1[8]/ENET_CRS
- net ETH_MDC: now also U2.P1[16]/ENET_MDC; no longer U7.P1[16]/ENET_MDC
- net ETH_MDIO: now also U2.P1[17]/ENET_MDIO; no longer U7.P1[17]/ENET_MDIO
- net ETH_RXD_0: now also U2.P1[9]/ENET_RXD0; no longer U7.P1[9]/ENET_RXD0
- net ETH_RXD_1: now also U2.P1[10]/ENET_RXD1; no longer U7.P1[10]/ENET_RXD1
- net ETH_RX_ER: now also U2.P1[14]/ENET_RX_ER; no longer U7.P1[14]/ENET_RX_ER
- net ETH_TXD_0: now also U2.P1[0]/ENET_TXD0; no longer U7.P1[0]/ENET_TXD0
- net ETH_TXD_1: now also U2.P1[1]/ENET_TXD1; no longer U7.P1[1]/ENET_TXD1
- net ETH_TXD_EN: now also U2.P1[4]/ENET_TX_EN; no longer U7.P1[4]/ENET_TX_EN
- net FAN_1_PWM: now also J8-1.S, U2.P2[0]/PWM1[1]/TXD1; no longer J7-1.S, U7.P2[0]/PWM1[1]/TXD1
- net FAN_1_SENSOR: now also J8-2.S, U2.P0[8]/I2STX_WS/MISO1/MAT2[2]; no longer J7-2.S, U7.P0[8]/I2STX_WS/MISO1/MAT2[2]
- net FAN_2_PWM: now also J8-3.S, U2.P2[1]/PWM1[2]/RXD1; no longer J7-3.S, U7.P2[1]/PWM1[2]/RXD1
- net FAN_2_SENSOR: now also J8-4.S, U2.P0[9]/I2STX_SDA/MOSI1/MAT2[3]; no longer J7-4.S, U7.P0[9]/I2STX_SDA/MOSI1/MAT2[3]
- net GND: now also C3.2, J1-2.S, J12-1.S, J13.5, U2.VREFN, U2.VSS, U2.VSSA, U2.VSS_2, U2.VSS_3, U2.VSS_4, U2.VSS_5, U2.VSS_6, U5.GND; no longer C115.2, U2.GND, U7.VREFN, U7.VSS, U7.VSSA, U7.VSS_2, U7.VSS_3, U7.VSS_4, U7.VSS_5, U7.VSS_6, X6.5
- net HMI_BUTTON_1: now also J10-1.S, R18.1; no longer J11-1.S, R13.1
- net HMI_BUTTON_2: now also J10-2.S, R19.1; no longer J11-2.S, R12.1
- net HMI_BUTTON_3: now also J10-3.S, R20.1; no longer J11-3.S, R11.1
- net HMI_BUTTON_4: now also J10-4.S, R21.1; no longer J11-4.S, R10.1
- net HMI_BUTTON_5: now also J10-5.S, R22.1; no longer J11-5.S, R9.1
- net HMI_BUTTON_6: now also J10-6.S, R23.1; no longer J11-6.S, R8.1
- net HMI_BUTTON_CPU_1: now also U2.P0[16]/RXD1/SSEL0/SSEL; no longer U7.P0[16]/RXD1/SSEL0/SSEL
- net HMI_BUTTON_CPU_2: now also U2.P0[15]/TXD1/SCK0/SCK; no longer U7.P0[15]/TXD1/SCK0/SCK
- net HMI_BUTTON_CPU_3: now also U2.P0[17]/CTS1/MISO0/MISO; no longer U7.P0[17]/CTS1/MISO0/MISO
- net HMI_BUTTON_CPU_4: now also U2.P0[18]/DCD1/MOSI0/MOSI, U5.1A; no longer U3.1A, U7.P0[18]/DCD1/MOSI0/MOSI
- net HMI_BUTTON_CPU_5: now also U2.P0[19]/DSR1/SDA1, U5.2A; no longer U3.2A, U7.P0[19]/DSR1/SDA1
- net HMI_BUTTON_CPU_6: now also R4.2, R5.1, U5.3A; no longer R16.2, R17.1, U3.3A
- net HMI_BUTTON_MCU_FCT_6: now also R5.2, U2.P0[20]/DTR1/SCL1; no longer R17.2, U7.P0[20]/DTR1/SCL1
- net HMI_LCD_BACKLIGHT: now also R13.2, U2.P0[22]/RTS1/TD1; no longer R15.2, U7.P0[22]/RTS1/TD1
- net HMI_LCD_LED+: now also J11-1.S, R11.2; no longer J12-1.S, R3.2
- net HMI_LCD_SCL: now also J11-2.S, R10.2, U2.P0[11]/RXD2/SCL2/MAT3[1], U3.SCL; no longer J12-2.S, R14.2, U2.SCL, U7.P0[11]/RXD2/SCL2/MAT3[1]
- net HMI_LCD_SDA: now also J11-3.S, R12.2, U2.P0[10]/TXD2/SDA2/MAT3[0], U3.SDA; no longer J12-3.S, R2.2, U2.SDA, U7.P0[10]/TXD2/SDA2/MAT3[0]
- net HMI_LCD_VO: now also J11-4.S, U3.W; no longer J12-4.S, U2.W
- net HMI_LED_1: now also R24.1, U2.P2[2]/PWM1[3]/CTS1/TRACEDATA[3]; no longer R7.1, U7.P2[2]/PWM1[3]/CTS1/TRACEDATA[3]
- net HMI_LED_2: now also R25.2, U2.P2[3]/PWM1[4]/DCD1/TRACEDATA[2]; no longer R6.2, U7.P2[3]/PWM1[4]/DCD1/TRACEDATA[2]
- net HMI_LED_3: now also R26.1, U2.P2[4]/PWM1[5]/DSR1/TRACEDATA[1]; no longer R5.1, U7.P2[4]/PWM1[5]/DSR1/TRACEDATA[1]
- net HMI_LED_4: now also R27.2, U2.P2[5]/PWM1[6]/DTR1/TRACEDATA[0]; no longer R4.2, U7.P2[5]/PWM1[6]/DTR1/TRACEDATA[0]
- net ISP_RXDO: now also J12-4.S, U2.P0[3]/RXD0/AD0[6]; no longer U7.P0[3]/RXD0/AD0[6]
- net ISP_TXDO: now also J12-5.S, U2.P0[2]/TXD0/AD0[7]; no longer U7.P0[2]/TXD0/AD0[7]
- net JTAG_TCK: now also U2.TCK/SWDCLK; no longer U7.TCK/SWDCLK
- net JTAG_TDI: now also U2.TDI; no longer U7.TDI
- net JTAG_TDO: now also U2.TDO/SWO; no longer U7.TDO/SWO
- net JTAG_TMS: now also U2.TMS/SWDIO; no longer U7.TMS/SWDIO
- net N$1: now also J14-2.S, R25.1; no longer J13-2.S, R6.1
- net N$15: now also J13.2, R15.1, R17.2; no longer R36.1, R38.2, X6.2
- net N$16: now also J13.3, R16.1; no longer R35.1, X6.3
- net N$17: now also R18.2; no longer R13.2
- net N$18: now also R14.1; no longer R39.1
- net N$19: now also R19.2; no longer R12.2
- net N$2: now also J14-4.S, R27.1; no longer J13-4.S, R4.1
- net N$20: now also R20.2; no longer R11.2
- net N$25: now also R21.2, U5.1Y; no longer R10.2, U3.1Y
- net N$26: now also R22.2, U5.2Y; no longer R9.2, U3.2Y
- net N$27: now also R23.2, U5.3Y; no longer R8.2, U3.3Y
- net N$5: now also R7.1, R8.2, R9.2; no longer R100.2, R101.2, R102.1
- net N$63: now also J14-1.S, R24.2; no longer J13-1.S, R7.2
- net N$64: now also J14-3.S, R26.2; no longer J13-3.S, R5.2
- net N$7: now also R13.1; no longer R15.1
- net RESET: now also R4.1, R6.1, U2.*RESET; no longer R103.1, R16.1, U7.*RESET
- net RTCX1: now also U2.RTCX1; no longer U7.RTCX1
- net RTCX2: now also U2.RTCX2; no longer U7.RTCX2
- net USB_D_N: now also R16.2, U2.P0[30]/USB_D?; no longer R35.2, U7.P0[30]/USB_D?
- net USB_D_P: now also R15.2, U2.P0[29]/USB_D+; no longer R36.2, U7.P0[29]/USB_D+
- net USB_UP_LED: now also R14.2, U2.P1[18]/USB_UP_LED/PWM1[1]/CAP1[0]; no longer R39.2, U7.P1[18]/USB_UP_LED/PWM1[1]/CAP1[0]
- net USB_V_BUS: now also J13.1, U2.P1[30]/VBUS/AD0[4]; no longer U7.P1[30]/VBUS/AD0[4], X6.1
- net VBAT+: now also U2.VBAT; no longer U7.VBAT
- net XTAL1: now also U2.XTAL1; no longer U7.XTAL1

Commit message: Add limitation resistance on Encoder output, ADC input, relay input and fan Add LED on board Poly for +5V on Route15
Parts:
- added LED2: (no value), led:LEDCHIPLED_0603
- added R28, R29, R30, R31, R32, R33, R34, R35, R36, R37, R38, R39, R40, R41: 100, rcl:R-EU_R0603
- added R42: 1K5, rcl:R-EU_R0603
Connections:
- new net !RESET: U2.*RESET
- new net LED_DEBUG: LED2.A, U2.P1[21]/*MCABORT/PWM1[3]/SSEL0
- new net N$10: J8-3.S, R34.1
- new net N$11: J8-4.S, R35.1
- new net N$12: J5-3.S, R37.1
- new net N$13: J5-2.S, R36.1
- new net N$14: J5-1.S, R31.1
- new net N$21: J6-4.S, R41.1
- new net N$23: J6-3.S, R40.1
- new net N$24: J6-2.S, R39.1
- new net N$28: J6-1.S, R38.1
- new net N$29: LED2.C, R42.1
- new net N$3: J7-1.S, R28.1
- new net N$4: J7-2.S, R29.1
- new net N$6: J7-3.S, R30.1
- new net N$8: J8-1.S, R32.1
- new net N$9: J8-2.S, R33.1
- net ADC_SLACK_DETECTION: now also R37.2; no longer J5-3.S
- net ADC_TEMP_0: now also R31.2; no longer J5-1.S
- net ADC_TEMP_1: now also R36.2; no longer J5-2.S
- net BRAKE_SENSOR_1: now also R38.2; no longer J6-1.S
- net BRAKE_SENSOR_2: now also R39.2; no longer J6-2.S
- net DRIVE_EN: now also R40.2; no longer J6-3.S
- net DRIVE_ERR: now also R41.2; no longer J6-4.S
- net ENCODER_A: now also R28.2; no longer J7-1.S
- net ENCODER_B: now also R29.2; no longer J7-2.S
- net ENCODER_Z: now also R30.2; no longer J7-3.S
- net FAN_1_PWM: now also R32.2; no longer J8-1.S
- net FAN_1_SENSOR: now also R33.2; no longer J8-2.S
- net FAN_2_PWM: now also R34.2; no longer J8-3.S
- net FAN_2_SENSOR: now also R35.2; no longer J8-4.S
- net GND: now also R42.2
- net RESET: no longer U2.*RESET

Commit message: Add pin name on the board
Parts:
- added JP2, JP3, JP4, JP5: FIDUCIAL1X2, SparkFun:FIDUCIAL1X2
- added T2: EXMACHINA-LOGO-NAME, exmachina:EXMACHINA-LOGO-NAME
- LED1, LED2: value (none) -> Blue
- R10: value 4K7 -> 1K5
- R11, R15, R16: value 33 -> 100
- R12: value 4K7 -> 100
- R14, R17, R42: value 1K5 -> 100
- R18, R19, R20, R21, R22, R23: value 1K -> 100
- R25, R27: value 100 -> 4K7
- R26, R30, R31: value 100 -> 33
- R29, R32: value 100 -> 1K5
- R33, R34, R35, R36, R37, R38: value 100 -> 1K
Connections:
- net +3V3: now also LED2.A, R25.1, R27.1, R32.1; no longer LED1.A, R10.1, R12.1, R17.1
- net +5V: now also R26.1; no longer R11.1
- net ADC_SLACK_DETECTION: now also R13.2; no longer R37.2
- net ADC_TEMP_0: now also R11.2; no longer R31.2
- net ADC_TEMP_1: now also R12.2; no longer R36.2
- net BRAKE_SENSOR_1: now also R17.2; no longer R38.2
- net BRAKE_SENSOR_2: now also R14.2; no longer R39.2
- net DRIVE_EN: now also R15.2; no longer R40.2
- net DRIVE_ERR: now also R16.2; no longer R41.2
- net ENCODER_A: now also R18.2; no longer R28.2
- net ENCODER_B: now also R19.2; no longer R29.2
- net ENCODER_Z: now also R20.2; no longer R30.2
- net FAN_1_PWM: now also R21.2; no longer R32.2
- net FAN_1_SENSOR: now also R22.2; no longer R33.2
- net FAN_2_PWM: now also R23.2; no longer R34.2
- net FAN_2_SENSOR: now also R24.2; no longer R35.2
- net GND: now also R10.2; no longer R42.2
- net HMI_BUTTON_1: now also R33.1; no longer R18.1
- net HMI_BUTTON_2: now also R34.1; no longer R19.1
- net HMI_BUTTON_3: now also R35.1; no longer R20.1
- net HMI_BUTTON_4: now also R36.1; no longer R21.1
- net HMI_BUTTON_5: now also R37.1; no longer R22.1
- net HMI_BUTTON_6: now also R38.1; no longer R23.1
- net HMI_LCD_BACKLIGHT: now also R28.2; no longer R13.2
- net HMI_LCD_LED+: now also R26.2; no longer R11.2
- net HMI_LCD_SCL: now also R25.2; no longer R10.2
- net HMI_LCD_SDA: now also R27.2; no longer R12.2
- net HMI_LED_1: now also R39.1; no longer R24.1
- net HMI_LED_2: now also R40.2; no longer R25.2
- net HMI_LED_3: now also R41.1; no longer R26.1
- net HMI_LED_4: now also R42.2; no longer R27.2
- net LED_DEBUG: now also LED1.A; no longer LED2.A
- net N$1: now also R40.1; no longer R25.1
- net N$10: now also R23.1; no longer R34.1
- net N$11: now also R24.1; no longer R35.1
- net N$12: now also R13.1; no longer R37.1
- net N$13: now also R12.1; no longer R36.1
- net N$14: now also R11.1; no longer R31.1
- net N$15: now also R30.1, R32.2; no longer R15.1, R17.2
- net N$16: now also R31.1; no longer R16.1
- net N$17: now also R33.2; no longer R18.2
- net N$18: now also LED2.C, R29.1; no longer LED1.C, R14.1
- net N$19: now also R34.2; no longer R19.2
- net N$2: now also R42.1; no longer R27.1
- net N$20: now also R35.2; no longer R20.2
- net N$21: now also R16.1; no longer R41.1
- net N$23: now also R15.1; no longer R40.1
- net N$24: now also R14.1; no longer R39.1
- net N$25: now also R36.2; no longer R21.2
- net N$26: now also R37.2; no longer R22.2
- net N$27: now also R38.2; no longer R23.2
- net N$28: now also R17.1; no longer R38.1
- net N$29: now also LED1.C, R10.1; no longer LED2.C, R42.1
- net N$3: now also R18.1; no longer R28.1
- net N$4: now also R19.1; no longer R29.1
- net N$6: now also R20.1; no longer R30.1
- net N$63: now also R39.2; no longer R24.2
- net N$64: now also R41.2; no longer R26.2
- net N$7: now also R28.1; no longer R13.1
- net N$8: now also R21.1; no longer R32.1
- net N$9: now also R22.1; no longer R33.1
- net USB_D_N: now also R31.2; no longer R16.2
- net USB_D_P: now also R30.2; no longer R15.2
- net USB_UP_LED: now also R29.2; no longer R14.2
Other:
- moved on the sheet: R11, R12, R13, R14, R15, R16, R17, R18, R19, R20, R21, R22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

Commit message: Generate gerber files and BOM and part list
Parts:
- C1: MPN (none) -> F931A106MAA; OC_NEWARK (none) -> 58R3260
- C10, C5: MPN (none) -> MC0603N180K500CT; OC_NEWARK (none) -> 06R5140
- C11, C12, C13, C14, C15, C16, C17, C18, C19, C2, C20, C21, C3, C4, C6, C7, C8, C9: MPN (none) -> MC0603B104K160CT; OC_NEWARK (none) -> 06R4923
- H1, H2, H3, H4, JP1, JP2, JP3, JP4, JP5, L1, SW1, SW2, T2: OC_NEWARK (none) -> unknown
- J1, J10, J2: MPN (none) -> 22-05-7068; OC_NEWARK (none) -> 25M1733
- J11, J14, J6, J8: MPN (none) -> 22-05-7048; OC_NEWARK (none) -> 26M6363
- J12: MF (none) -> MOLEX; MPN (none) -> 22-27-2061; OC_NEWARK (none) -> 56H0719
- J13: MPN (none) -> USB3075-30-A; OC_NEWARK (none) -> 58T0863
- J15: MPN (none) -> 1241050-5; OC_NEWARK (none) -> 98K5467
- J3, J9: MPN (none) -> 22-05-7028; OC_NEWARK (none) -> 25M1728
- J4: value 22-05-7028-02 -> 22-05-7038-03; device con-molex:22-05-7028-02 -> con-molex:22-05-7038-03; MPN (none) -> 22-05-7038; OC_NEWARK (none) -> 26M6362
- J5, J7: MPN (none) -> 22-05-7038; OC_NEWARK (none) -> 26M6362
- LED1, LED2: MPN (none) -> OVS-0603; OC_NEWARK (none) -> 15R2205
- R1, R2, R25, R27, R3: MPN (none) -> MCMR06X4701FTL; OC_NEWARK (none) -> 86T3649
- R10, R29, R32: MPN (none) -> MCMR06X1501FTL; OC_NEWARK (none) -> 86T3542
- R11, R12, R13, R14, R15, R16, R17, R18, R19, R20, R21, R22, R23, R24, R28, R39, R40, R41, R42: MPN (none) -> MCMR06X1000FTL; OC_NEWARK (none) -> 86T3504
- R26, R30, R31: MPN (none) -> MCMR06X33R0FTL; OC_NEWARK (none) -> 86T3614
- R33, R34, R35, R36, R37, R38: MPN (none) -> MCMR06X1001FTL; OC_NEWARK (none) -> 86T3505
- R4, R5, R8, R9: MPN (none) -> MCMR06X000 PTL; OC_NEWARK (none) -> 86T3500
- R6, R7: MPN (none) -> MCMR06X1002FTL; OC_NEWARK (none) -> 86T3506
- T1: MF (none) -> ON SEMICONDUCTOR; MPN (none) -> MMBT2222ALT1G; OC_NEWARK (none) -> 84K8795
- U2: MPN (none) -> LPC1768FBD100; OC_NEWARK (none) -> 15R1840
- U3: MPN (none) -> ISL90728WIE627Z-TK; OC_NEWARK (none) -> 65T7357
- U4, U5: MF (none) -> TEXAS INSTRUMENTS
- X1: MPN (none) -> Q13FC13500004; OC_NEWARK (none) -> 31M4970
- X2: MPN (none) -> ASE-12.000MHZ-LC-T; OC_NEWARK (none) -> 40Y2118
- X3: MF (none) -> KEYSTONE ELECTR; MPN (none) -> 3000; OC_NEWARK (none) -> 66F5622
Connections:
- net +3V3: now also J4-2.S; no longer J4-1.S
- net AVDD: now also J4-1.S
- net GND: now also J4-3.S; no longer J4-2.S
Other:
- moved on the sheet: J3-1, J3-2, J4-1, J4-2
